File: pcb-left/pcb-left.sch (KiCad schematic (older format))
At the start: 80 parts

Commit message: added pcb files
Parts:
- C1, C2, C3, C4, C5, C6, C7: renamed from C?; footprint (none) -> Capacitor_SMD:C_0805_2012Metric
- D1, D10, D11, D12, D13, D14, D15, D16, D17, D18, D19, D2, D20, D21, D22, D23, D24, D25, D26, D27, D28, D29, D3, D30, D4, D5, D6, D7, D8, D9: renamed from D?; footprint (none) -> Diode_SMD:D_SOD-123
- MX1, MX11, MX12, MX13, MX14, MX16, MX17, MX18, MX19, MX21, MX22, MX23, MX24, MX26, MX27, MX28, MX29, MX30, MX6, MX7, MX8, MX9: renamed from MX?; footprint (none) -> MX_Alps_Hybrid:MXOnly-1U-NoLED
- MX10, MX15, MX25, MX5: renamed from MX?; footprint (none) -> MX_Alps_Hybrid:MXOnly-1.25U-NoLED
- MX2: renamed from MX?; footprint (none) -> MX_Alps_Hybrid:MXOnly-1.5U-NoLED
- MX20, MX4: renamed from MX?; footprint (none) -> MX_Alps_Hybrid:MXOnly-2.25U-NoLED
- MX3: renamed from MX?; footprint (none) -> MX_Alps_Hybrid:MXOnly-1.75U-NoLED
- R1, R2, R3, R4, R5, R6, R7, R8: renamed from R?; footprint (none) -> Resistor_SMD:R_0805_2012Metric
- SW1: renamed from SW?; footprint (none) -> random-keyboard-parts:SKQG-1155865
- USB1, USB2: renamed from USB?; footprint (none) -> Keebio-Parts:HRO-TYPE-C-31-M-12-Assembly
- Y1: renamed from Y?; footprint (none) -> Crystal:Crystal_SMD_3225-4Pin_3.2x2.5mm
- gave numbers to parts that had none: 1
Connections:
- net GND: now also USB1.1 (GND), USB1.12 (GND)

Commit message: finished left side pcb
Connections:
- net +5V: now also USB1.11 (VBUS), USB1.2 (VBUS)
- net GND: now also USB1.13 (SHIELD), USB2.13 (SHIELD)
- net SD+: now also U1.18 (PD0)
- net SD-: now also U1.19 (PD1)
- net col0: now also U1.31 (PC6)
- net col1: now also U1.37 (PF6)
- net col2: now also U1.36 (PF7)
- net col3: now also U1.20 (PD2)
- net col4: now also U1.21 (PD3)
- net col5: now also U1.22 (PD5)
- net col6: now also U1.12 (PB7)
- net row0: now also U1.8 (PB0)
- net row1: now also U1.11 (PB3)
- net row2: now also U1.10 (PB2)
- net row3: now also U1.9 (PB1)
- net row4: now also U1.29 (PB5)
Changed lines of the file:
@@
 $EndComp
 Connection ~ 1600 6300
+Text GLabel 10450 3550 2    50   Input ~ 0
+SD+
+Text GLabel 10450 3650 2    50   Input ~ 0
+SD-
+Text GLabel 10450 2850 2    50   Input ~ 0
+row4
+Text GLabel 10450 2450 2    50   Input ~ 0
+row3
+Text GLabel 10450 2550 2    50   Input ~ 0
+row2
+Text GLabel 10450 2650 2    50   Input ~ 0
+row1
+Text GLabel 10450 2350 2    50   Input ~ 0
+row0
+Text GLabel 10450 5250 2    50   Input ~ 0
+col2
+Text GLabel 10450 5150 2    50   Input ~ 0
+col1
+Text GLabel 10450 3250 2    50   Input ~ 0
+col0
+Text GLabel 10450 3750 2    50   Input ~ 0
+col3
+Text GLabel 10450 3850 2    50   Input ~ 0
+col4
+Text GLabel 10450 4050 2    50   Input ~ 0
+col5
+Text GLabel 10450 3050 2    50   Input ~ 0
+col6
+$Comp
+L power:+5V #PWR0115
+U 1 1 62B44302
+P 1650 5300
+F 0 "#PWR0115" H 1650 5150 50  0001 C CNN
+F 1 "+5V" H 1665 5473 50  0000 C CNN
+F 2 "" H 1650 5300 50  0001 C CNN
+F 3 "" H 1650 5300 50  0001 C CNN
+	1    1650 5300
+	1    0    0    -1
+$EndComp
+Connection ~ 1650 5300
+Wire Wire Line
+	1450 6400 1600 6400
+Wire Wire Line
+	1600 6400 1600 6300
+Wire Wire Line
+	3300 6400 3450 6400
+Wire Wire Line
+	3450 6400 3450 6300
+Connection ~ 3450 6300
 $EndSCHEMATC

Commit message: finalized left side pcb
Parts:
- added R9: 10k, Resistor_SMD:R_0805_2012Metric, symbol Device:R_Small
Connections:
- net +5V: now also R9.1
- net at U1.1 (PE6): now also R9.2
Changed lines of the file:
@@
 	3450 6400 3450 6300
 Connection ~ 3450 6300
+$Comp
+L Device:R_Small R9
+U 1 1 62ACB3C6
+P 10550 4550
+F 0 "R9" V 10354 4550 50  0000 C CNN
+F 1 "10k" V 10445 4550 50  0000 C CNN
+F 2 "Resistor_SMD:R_0805_2012Metric" H 10550 4550 50  0001 C CNN
+F 3 "~" H 10550 4550 50  0001 C CNN
+	1    10550 4550
+	0    1    1    0
+$EndComp
+$Comp
+L power:+5V #PWR0116
+U 1 1 62ACC0D8
+P 10650 4550
+F 0 "#PWR0116" H 10650 4400 50  0001 C CNN
+F 1 "+5V" H 10665 4723 50  0000 C CNN
+F 2 "" H 10650 4550 50  0001 C CNN
+F 3 "" H 10650 4550 50  0001 C CNN
+	1    10650 4550
+	1    0    0    -1
+$EndComp
 $EndSCHEMATC
